Commit message: Update rosbot.xacro

File: src/rosbot_description/urdf/rosbot.xacro (robot description, xacro)
@@ -60,5 +60,5 @@
         <mesh filename="package://rosbot_description/meshes/upper.stl" scale="0.001 0.001 0.001" />
       </geometry>
-      <material name="Red"/>
+      <material name="Blue"/>
     </visual>
   </link>
